File: ArduinoTrack Flex/Flex.brd (EAGLE design)
At the start: 67.3 x 85.7 mm, 64 parts, among them J1 5.5x2.1mm Barrel, Q1 BSS138, Q2 2N2222, U2 UBLOX_MAX, U3 LM1086, U4 RADIOMETRIX-HX1-CUSTOM, U5 LP3985IM5-3.3/NOPB, U6 MCP6L01T, U7 ATMega328, U8 BME280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

Commit message: Fixed alignment for transmitter board
Shifted piezo down, and SMA up to make room for transmitter board.
Parts:
- D1, D2: device diode:SOD123 -> custom-ds:SOD123
- moved R8 2.86 mm to (28.6, 43.2)
- moved X1 2.54 mm to (39.7, 83.2)
- moved LED1 2.54 mm to (29.2, 84.5)
- moved LED2 2.54 mm to (31.8, 84.5)
- moved SG1 0.95 mm to (45.1, 37.8)
Connections:
- net XCEIVER-RX: now also U7.13; no longer U7.14
- net XCEIVER-TX: now also U7.14; no longer U7.13
Routing:
- net AUD-ANNUNC: track 33.3 -> 29.9 mm
- net N$27: track 3.07 -> 5.93 mm
- net N$4: track 5.71 -> 8.25 mm
- net N$25: track 88.4 -> 90.9 mm
- net N$23: track 3.70 -> 6.24 mm
- net N$9: track 20.3 -> 21.6 mm
Other:
- board size 67.3 x 85.7 mm -> 67.3 x 88.9 mm
- board text added: "ArduinoTrack Flex v1.02 Custom Digital Services, LLC www.custom-ds.com"
- board text removed: "ArduinoTrack Flex v1.01 Custom Digital Services, LLC www.custom-ds.com"
