File: ArduinoTrack Flex/Flex.sch (EAGLE design)
At the start: 64 parts, among them J1 5.5x2.1mm Barrel, Q1 BSS138, Q2 2N2222, U2 UBLOX_MAX, U3 LM1086, U4 RADIOMETRIX-HX1-CUSTOM, U5 LP3985IM5-3.3/NOPB, U6 MCP6L01T, U7 ATMega328, U8 BME280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

Commit message: Fixed alignment for transmitter board
Shifted piezo down, and SMA up to make room for transmitter board.
Parts:
- D1, D2: device diode:DIODE-SOD123 -> custom-ds:DIODE-SOD123
Connections:
- net XCEIVER-RX: now also U7.PB1(OC1A); no longer U7.PB2(SS/OC1B)
- net XCEIVER-TX: now also U7.PB2(SS/OC1B); no longer U7.PB1(OC1A)
Changed lines of the file:
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@@
 <attribute name="DIGIKEY" value="MCP6L01T-E/OTCT-ND"/>
 </part>
-<part name="D2" library="diode" deviceset="DIODE-" device="SOD123" value="1N4148W">
+<part name="D2" library="custom-ds" deviceset="DIODE-" device="SOD123" value="1N4148W">
 <attribute name="DIGIKEY" value="1N4148W-FDICT-ND"/>
 </part>
@@
 <part name="GND7" library="supply1" deviceset="GND" device=""/>
 <part name="P+3" library="supply1" deviceset="+5V" device=""/>
-<part name="D1" library="diode" deviceset="DIODE-" device="SOD123" value="1N4148W">
+<part name="D1" library="custom-ds" deviceset="DIODE-" device="SOD123" value="1N4148W">
 <attribute name="DIGIKEY" value="1N4148W-FDICT-ND"/>
 </part>
@@
 <net name="XCEIVER-TX" class="0">
 <segment>
-<pinref part="U7" gate="G$1" pin="PB1(OC1A)"/>
-<wire x1="99.06" y1="127" x2="101.6" y2="127" width="0.1524" layer="91"/>
-<label x="101.6" y="127" size="1.27" layer="95" xref="yes"/>
+<wire x1="99.06" y1="124.46" x2="101.6" y2="124.46" width="0.1524" layer="91"/>
+<label x="101.6" y="124.46" size="1.27" layer="95" xref="yes"/>
+<pinref part="U7" gate="G$1" pin="PB2(SS/OC1B)"/>
 </segment>
 <segment>
@@
 <net name="XCEIVER-RX" class="0">
 <segment>
-<pinref part="U7" gate="G$1" pin="PB2(SS/OC1B)"/>
-<wire x1="99.06" y1="124.46" x2="101.6" y2="124.46" width="0.1524" layer="91"/>
-<label x="101.6" y="124.46" size="1.27" layer="95" xref="yes"/>
+<wire x1="99.06" y1="127" x2="101.6" y2="127" width="0.1524" layer="91"/>
+<label x="101.6" y="127" size="1.27" layer="95" xref="yes"/>
+<pinref part="U7" gate="G$1" pin="PB1(OC1A)"/>
 </segment>
 <segment>
@@
 </sheet>
 </sheets>
-<errors>
-</errors>
 </schematic>
 </drawing>
