File: ptFlex/ptFlex.sch (EAGLE design)
At the start: 64 parts, among them J1 5.5x2.1mm Barrel, Q1 BSS138, Q2 2N2222, U2 UBLOX_MAX, U3 LM1086, U4 RADIOMETRIX-HX1-CUSTOM, U5 LP3985IM5-3.3/NOPB, U6 MCP6L01T, U7 ATMega328, U8 BME280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

Commit message: Added digikey part numbers to missing parts.
Parts:
- SV2: DIGIKEY (none) -> 455-1804-1-ND
- U8: DIGIKEY (none) -> 828-1063-1-ND
Changed lines of the file:
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@@
 <attribute name="DIGIKEY" value="1N4148W-FDICT-ND"/>
 </part>
-<part name="SV2" library="SparkFun-Connectors" deviceset="I2C_STANDARD" device="QWIIC" value="Qwiic Right Angle"/>
+<part name="SV2" library="SparkFun-Connectors" deviceset="I2C_STANDARD" device="QWIIC" value="Qwiic Right Angle">
+<attribute name="DIGIKEY" value="455-1804-1-ND"/>
+</part>
 <part name="GND18" library="supply1" deviceset="GND" device=""/>
-<part name="U8" library="SparkFun-Sensors" deviceset="BME280" device="" value="BME280"/>
+<part name="U8" library="SparkFun-Sensors" deviceset="BME280" device="" value="BME280">
+<attribute name="DIGIKEY" value="828-1063-1-ND"/>
+</part>
 </parts>
 <sheets>
@@
 <attribute name="DIGIKEY" x="45.72" y="185.42" size="1.778" layer="96" rot="R90" display="off"/>
 </instance>
-<instance part="SV2" gate="G$1" x="175.26" y="167.64" rot="R270"/>
+<instance part="SV2" gate="G$1" x="175.26" y="167.64" rot="R270">
+<attribute name="DIGIKEY" x="175.26" y="167.64" size="1.778" layer="96" rot="R270" display="off"/>
+</instance>
 <instance part="GND18" gate="1" x="172.72" y="149.86"/>
-<instance part="U8" gate="U1" x="33.02" y="50.8"/>
+<instance part="U8" gate="U1" x="33.02" y="50.8">
+<attribute name="DIGIKEY" x="33.02" y="50.8" size="1.778" layer="96" display="off"/>
+</instance>
 </instances>
 <busses>

Commit message: Added GPS filter
Version 1.04
Parts:
- added F1: MURATA-GPS-FILTER, custom-ds:MURATA-GPS-FILTER
- renumbered SV1 to J3, SV2 to J4, SV3 to J2
Connections:
- removed net N$16: ANT1.FEED, U2.11_RF_IN
- new net N$2: F1.RF-1, U2.11_RF_IN
- new net N$3: ANT1.FEED, F1.RF-3
- net GND: now also F1.GND2, F1.GND4
Other:
- moved on the sheet: ANT1, C10, C11, C12, C13, C14, C15, C16, C17, C6, C7, C8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

Commit message: Final check in for hardware version 1
Parts:
- removed L4, L5, L6, L7: 160 ohm, inductor-neosid:SM-1206
- removed U4: RADIOMETRIX-HX1-CUSTOM, custom-ds:RADIOMETRIX-HX1-CUSTOM
- added C18, C19, C20, C21: .1uF, resistor:C-USC0805
- added D4: LL4148, custom-ds:LL4148
- added Q3: BSS138, SparkFun-DiscreteSemi:MOSFET-NCHANNELBSS138
- added R18, R19, R20, R21, R22, R23, R24, R25, R26: 10k, resistor:R-US_R0805
- added U1: DRA818V, custom-ds:DRA818V
- L1, L2, L3: value 160 ohm -> 1µH; device inductor-neosid:SM-1206 -> custom-ds:INDUCTOR; DIGIKEY 240-2411-1-ND -> (none)
Connections:
- removed net N$23: LED1.A, R5.2
- removed net RFGND: U4.ANTENNA_GND1, U4.ANTENNA_GND2, X1.2
- removed net VCC: L7.1, U4.VCC
- new net N$16: R19.1, R20.2, U1.PD
- new net N$21: LED1.C, R5.2
- new net N$28: R26.1, U1.RXD
- new net N$6: C18.1, L1.1, U1.ANT
- net +5V: now also D4.ANODE, LED1.A, R24.2; no longer L7.2
- net DIG-PTT: now also R18.1; no longer L1.2
- net DIG-XMIT-PS: now also R20.1; no longer L2.1
- net GND: now also C18.2, C19.2, C20.2, C21.2, R19.2, R21.2, R22.2, R23.1, U1.GND_1, U1.GND_2, X1.2; no longer LED1.C, U4.GND
- net N$10: now also U1.MIC_IN; no longer L4.2
- net N$12: now also D4.CATHODE, Q3.G, R25.2, U1.VBAT; no longer L5.2, U4.RX_AUDIO
- net N$14: now also R18.2, R21.1, U1.PTT; no longer L2.2, U4.POWER_SAVE
- net N$19: now also R22.1, U1.H/L; no longer L6.2, U4.RX_DATA
- net N$20: now also Q3.S, R25.1, U1.TXD; no longer L3.2, U4.TX_DATA
- net N$4: now also C20.1, L2.2, L3.1; no longer U4.ANTENNA, X1.1
- net N$5: now also C19.1, L1.2, L2.1; no longer L4.1, U4.TX_AUDIO
- net N$7: now also C21.1, L3.2, X1.1; no longer L1.1, U4.PTT
- net RX-AUDIO: now also U1.AF_OUT; no longer L5.1
- net XCEIVER-RX: now also R23.2, R26.2; no longer L3.1
- net XCEIVER-TX: now also Q3.D, R24.1; no longer L6.1
Other:
- moved on the sheet: LED1, X1
